File: DnD_Puzzle_1/schema.sch (EAGLE design)
At the start: 13 parts, among them IC1 MEGA32-P

Commit message: working on the electronic scheme
Parts:
- added T1, T2, T3: (no value), transistor:-PNP-TO92
Connections:
- new net N$1: IC1.(TOSC2)PC7, R8.1
- new net N$2: IC1.(TOSC1)PC6, R7.1
- new net N$3: IC1.(TDI)PC5, R6.1
- new net N$4: IC1.(TDO)PC4, R5.1
- new net N$5: IC1.(TMS)PC3, R4.1
- new net N$6: IC1.(TCK)PC2, R3.1
- new net N$7: IC1.(SDA)PC1, R2.1
- new net N$8: IC1.(SCL)PC0, R1.1
Other:
- moved on the sheet: R1, R10, R11, R12, R2, R3, R4, R5, R6, R7, R8, R9
Changed lines of the file:
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@@
 <part name="R11" library="resistor-power" library_urn="urn:adsk.eagle:library:344" deviceset="R" device="AC01" package3d_urn="urn:adsk.eagle:package:25124/1"/>
 <part name="R12" library="resistor-power" library_urn="urn:adsk.eagle:library:344" deviceset="R" device="AC01" package3d_urn="urn:adsk.eagle:package:25124/1"/>
+<part name="T1" library="transistor" library_urn="urn:adsk.eagle:library:402" deviceset="*-PNP-" device="TO92" package3d_urn="urn:adsk.eagle:package:28523/2"/>
+<part name="T2" library="transistor" library_urn="urn:adsk.eagle:library:402" deviceset="*-PNP-" device="TO92" package3d_urn="urn:adsk.eagle:package:28523/2"/>
+<part name="T3" library="transistor" library_urn="urn:adsk.eagle:library:402" deviceset="*-PNP-" device="TO92" package3d_urn="urn:adsk.eagle:package:28523/2"/>
 </parts>
 <sheets>
@@
 <attribute name="VALUE" x="0" y="-2.54" size="1.778" layer="96"/>
 </instance>
-<instance part="R1" gate="G$1" x="76.2" y="86.36" smashed="yes">
-<attribute name="NAME" x="72.39" y="87.7316" size="1.778" layer="95"/>
-<attribute name="VALUE" x="72.39" y="83.439" size="1.778" layer="96"/>
+<instance part="R1" gate="G$1" x="53.34" y="25.4" smashed="yes">
+<attribute name="NAME" x="45.974" y="26.0096" size="1.778" layer="95"/>
+<attribute name="VALUE" x="49.53" y="22.479" size="1.778" layer="96"/>
 </instance>
-<instance part="R2" gate="G$1" x="76.2" y="81.28" smashed="yes">
-<attribute name="NAME" x="72.39" y="82.6516" size="1.778" layer="95"/>
-<attribute name="VALUE" x="72.39" y="78.359" size="1.778" layer="96"/>
+<instance part="R2" gate="G$1" x="53.34" y="27.94" smashed="yes">
+<attribute name="NAME" x="45.974" y="28.5496" size="1.778" layer="95"/>
+<attribute name="VALUE" x="49.53" y="25.019" size="1.778" layer="96"/>
 </instance>
-<instance part="R3" gate="G$1" x="76.2" y="76.2" smashed="yes">
-<attribute name="NAME" x="72.39" y="77.5716" size="1.778" layer="95"/>
-<attribute name="VALUE" x="72.39" y="73.279" size="1.778" layer="96"/>
+<instance part="R3" gate="G$1" x="53.34" y="30.48" smashed="yes">
+<attribute name="NAME" x="45.974" y="31.0896" size="1.778" layer="95"/>
+<attribute name="VALUE" x="49.53" y="27.559" size="1.778" layer="96"/>
 </instance>
-<instance part="R4" gate="G$1" x="76.2" y="71.12" smashed="yes">
-<attribute name="NAME" x="72.39" y="72.4916" size="1.778" layer="95"/>
-<attribute name="VALUE" x="72.39" y="68.199" size="1.778" layer="96"/>
+<instance part="R4" gate="G$1" x="53.34" y="33.02" smashed="yes">
+<attribute name="NAME" x="45.974" y="33.6296" size="1.778" layer="95"/>
+<attribute name="VALUE" x="49.53" y="30.099" size="1.778" layer="96"/>
 </instance>
-<instance part="R5" gate="G$1" x="76.2" y="66.04" smashed="yes">
-<attribute name="NAME" x="72.39" y="67.4116" size="1.778" layer="95"/>
-<attribute name="VALUE" x="72.39" y="63.119" size="1.778" layer="96"/>
+<instance part="R5" gate="G$1" x="53.34" y="35.56" smashed="yes">
+<attribute name="NAME" x="45.974" y="35.9156" size="1.778" layer="95"/>
+<attribute name="VALUE" x="49.53" y="32.639" size="1.778" layer="96"/>
 </instance>
-<instance part="R6" gate="G$1" x="76.2" y="60.96" smashed="yes">
-<attribute name="NAME" x="72.39" y="62.3316" size="1.778" layer="95"/>
-<attribute name="VALUE" x="72.39" y="58.039" size="1.778" layer="96"/>
+<instance part="R6" gate="G$1" x="53.34" y="38.1" smashed="yes">
+<attribute name="NAME" x="45.974" y="38.4556" size="1.778" layer="95"/>
+<attribute name="VALUE" x="49.53" y="35.179" size="1.778" layer="96"/>
 </instance>
-<instance part="R7" gate="G$1" x="76.2" y="55.88" smashed="yes">
-<attribute name="NAME" x="72.39" y="57.2516" size="1.778" layer="95"/>
-<attribute name="VALUE" x="72.39" y="52.959" size="1.778" layer="96"/>
+<instance part="R7" gate="G$1" x="53.34" y="40.64" smashed="yes">
+<attribute name="NAME" x="45.974" y="40.9956" size="1.778" layer="95"/>
+<attribute name="VALUE" x="49.53" y="37.719" size="1.778" layer="96"/>
 </instance>
-<instance part="R8" gate="G$1" x="76.2" y="50.8" smashed="yes">
-<attribute name="NAME" x="72.39" y="52.1716" size="1.778" layer="95"/>
-<attribute name="VALUE" x="72.39" y="47.879" size="1.778" layer="96"/>
+<instance part="R8" gate="G$1" x="53.34" y="43.18" smashed="yes">
+<attribute name="NAME" x="45.974" y="43.5356" size="1.778" layer="95"/>
+<attribute name="VALUE" x="49.53" y="40.259" size="1.778" layer="96"/>
 </instance>
-<instance part="R9" gate="G$1" x="78.74" y="45.72" smashed="yes">
-<attribute name="NAME" x="74.93" y="47.0916" size="1.778" layer="95"/>
-<attribute name="VALUE" x="74.93" y="42.799" size="1.778" layer="96"/>
+<instance part="R9" gate="G$1" x="116.84" y="58.42" smashed="yes">
+<attribute name="NAME" x="113.03" y="59.7916" size="1.778" layer="95"/>
+<attribute name="VALUE" x="113.03" y="55.499" size="1.778" layer="96"/>
 </instance>
-<instance part="R10" gate="G$1" x="78.74" y="40.64" smashed="yes">
-<attribute name="NAME" x="74.93" y="42.0116" size="1.778" layer="95"/>
-<attribute name="VALUE" x="74.93" y="37.719" size="1.778" layer="96"/>
+<instance part="R10" gate="G$1" x="116.84" y="53.34" smashed="yes">
+<attribute name="NAME" x="113.03" y="54.7116" size="1.778" layer="95"/>
+<attribute name="VALUE" x="113.03" y="50.419" size="1.778" layer="96"/>
 </instance>
-<instance part="R11" gate="G$1" x="78.74" y="35.56" smashed="yes">
-<attribute name="NAME" x="74.93" y="36.9316" size="1.778" layer="95"/>
-<attribute name="VALUE" x="74.93" y="32.639" size="1.778" layer="96"/>
+<instance part="R11" gate="G$1" x="116.84" y="48.26" smashed="yes">
+<attribute name="NAME" x="113.03" y="49.6316" size="1.778" layer="95"/>
+<attribute name="VALUE" x="113.03" y="45.339" size="1.778" layer="96"/>
 </instance>
-<instance part="R12" gate="G$1" x="78.74" y="30.48" smashed="yes">
-<attribute name="NAME" x="74.93" y="31.8516" size="1.778" layer="95"/>
-<attribute name="VALUE" x="74.93" y="27.559" size="1.778" layer="96"/>
+<instance part="R12" gate="G$1" x="119.38" y="43.18" smashed="yes">
+<attribute name="NAME" x="115.57" y="44.5516" size="1.778" layer="95"/>
+<attribute name="VALUE" x="115.57" y="40.259" size="1.778" layer="96"/>
+</instance>
+<instance part="T1" gate="G$1" x="101.6" y="53.34" smashed="yes">
+<attribute name="NAME" x="91.44" y="60.96" size="1.778" layer="95"/>
+<attribute name="VALUE" x="91.44" y="58.42" size="1.778" layer="96"/>
+</instance>
+<instance part="T2" gate="G$1" x="101.6" y="35.56" smashed="yes">
+<attribute name="NAME" x="91.44" y="43.18" size="1.778" layer="95"/>
+<attribute name="VALUE" x="91.44" y="40.64" size="1.778" layer="96"/>
+</instance>
+<instance part="T3" gate="G$1" x="101.6" y="17.78" smashed="yes">
+<attribute name="NAME" x="91.44" y="25.4" size="1.778" layer="95"/>
+<attribute name="VALUE" x="91.44" y="22.86" size="1.778" layer="96"/>
 </instance>
 </instances>
@@
 </busses>
 <nets>
+<net name="N$1" class="0">
+<segment>
+<pinref part="IC1" gate="G$1" pin="(TOSC2)PC7"/>
+<pinref part="R8" gate="G$1" pin="1"/>
+<wire x1="35.56" y1="43.18" x2="48.26" y2="43.18" width="0.1524" layer="91"/>
+</segment>
+</net>
+<net name="N$2" class="0">
+<segment>
+<pinref part="IC1" gate="G$1" pin="(TOSC1)PC6"/>
+<pinref part="R7" gate="G$1" pin="1"/>
+<wire x1="35.56" y1="40.64" x2="48.26" y2="40.64" width="0.1524" layer="91"/>
+</segment>
+</net>
+<net name="N$3" class="0">
+<segment>
+<pinref part="IC1" gate="G$1" pin="(TDI)PC5"/>
+<pinref part="R6" gate="G$1" pin="1"/>
+<wire x1="35.56" y1="38.1" x2="48.26" y2="38.1" width="0.1524" layer="91"/>
+</segment>
+</net>
+<net name="N$4" class="0">
+<segment>
+<pinref part="IC1" gate="G$1" pin="(TDO)PC4"/>
+<pinref part="R5" gate="G$1" pin="1"/>
+<wire x1="35.56" y1="35.56" x2="48.26" y2="35.56" width="0.1524" layer="91"/>
+</segment>
+</net>
+<net name="N$5" class="0">
+<segment>
+<pinref part="IC1" gate="G$1" pin="(TMS)PC3"/>
+<pinref part="R4" gate="G$1" pin="1"/>
+<wire x1="35.56" y1="33.02" x2="48.26" y2="33.02" width="0.1524" layer="91"/>
+</segment>
+</net>
+<net name="N$6" class="0">
+<segment>
+<pinref part="IC1" gate="G$1" pin="(TCK)PC2"/>
+<pinref part="R3" gate="G$1" pin="1"/>
+<wire x1="35.56" y1="30.48" x2="48.26" y2="30.48" width="0.1524" layer="91"/>
+</segment>
+</net>
+<net name="N$7" class="0">
+<segment>
+<pinref part="IC1" gate="G$1" pin="(SDA)PC1"/>
+<pinref part="R2" gate="G$1" pin="1"/>
+<wire x1="35.56" y1="27.94" x2="48.26" y2="27.94" width="0.1524" layer="91"/>
+</segment>
+</net>
+<net name="N$8" class="0">
+<segment>
+<pinref part="IC1" gate="G$1" pin="(SCL)PC0"/>
+<pinref part="R1" gate="G$1" pin="1"/>
+<wire x1="35.56" y1="25.4" x2="48.26" y2="25.4" width="0.1524" layer="91"/>
+</segment>
+</net>
 </nets>
 </sheet>

Commit message: working on the electronic scheme
Parts:
- added LED1, LED2, LED3, LED4: LA-401AN, led-7-segment:LA-401AN
- added T4: (no value), transistor:-PNP-TO92
Connections:
- new net N$10: IC1.(ADC1)PA1, R10.1
- new net N$11: IC1.(ADC2)PA2, R11.1
- new net N$12: IC1.(ADC3)PA3, R12.1
- new net N$13: R12.2, T1.B
- new net N$14: R11.2, T2.B
- new net N$15: R10.2, T3.B
- new net N$16: R9.2, T4.B
- new net N$9: IC1.(ADC0)PA0, R9.1
Other:
- moved on the sheet: R1, R10, R11, R12, R2, R3, R4, R5, R6, R7, R8, R9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

Commit message: Electronic schema finshed
Parts:
- R1, R2, R3, R4, R5, R6, R7, R8: value (none) -> 100R
- R10, R11, R12, R9: value (none) -> 2.2k
- T1, T2, T3, T4: value (none) -> BC559C
Connections:
- new net A: LED1.A, LED2.A, LED3.A, LED4.A, R1.2
- new net ANODE1: LED1.C@1, LED1.C@2, T4.C
- new net ANODE2: LED2.C@1, LED2.C@2, T3.C
- new net ANODE3: LED3.C@1, LED3.C@2, T2.C
- new net ANODE4: LED4.C@1, LED4.C@2, T1.C
- new net B: LED1.B, LED2.B, LED3.B, LED4.B, R2.2
- new net C: LED1.C, LED2.C, LED3.C, LED4.C, R3.2
- new net D: LED1.D, LED2.D, LED3.D, LED4.D, R4.2
- new net DP: LED1.DP, LED2.DP, LED3.DP, LED4.DP, R8.2
- new net E: LED1.E, LED2.E, LED3.E, LED4.E, R5.2
- new net F: LED1.F, LED2.F, LED3.F, LED4.F, R6.2
- new net G: LED1.G, LED2.G, LED3.G, LED4.G, R7.2
- new net VCC: T1.E, T2.E, T3.E, T4.E
Other:
- note added: "FJ5461BH used - 4 digits LED display"
- note added: "Schema without power supply of microcontroller!"
- moved on the sheet: LED1, LED2, LED3, LED4, R1, R2, R3, R4, R5, R6, R7, R8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

Commit message: schema.pdf updated
Parts:
- added D1: LED, ngspice-simulation:LED
- added R13, R15, R17, R19: 2.2k, resistor-power:RAC01
- added R14, R18: 10k, resistor-power:RAC01
- added R16: 220R, resistor-power:RAC01
- added S1: 5511, switch:5511
- added SP1: AL11P, buzzer:AL11P
- added T10, T6, T7, T9: BC337, transistor:2N2405
- added T5, T8: L-53P3C, opto-trans-siemens:BP103
Connections:
- new net GND: S1.NC, S1.NO, T10.E, T6.E, T7.E, T9.E
- new net N$17: R13.2, T5.E
- new net N$18: R13.1, T6.B
- new net N$19: R17.1, T9.B
- new net N$20: R15.1, T7.B
- new net N$21: IC1.(RXD)PD0, SP1.1
- new net N$22: IC1.(T1)PB1, S1.1A, S1.1B
- new net N$23: R14.2, R15.2, T6.C
- new net N$24: R17.2, T8.E
- new net N$25: R16.1, T10.C
- new net N$26: R18.2, R19.2, T9.C
- new net N$27: D1.A, R16.2
- new net N$28: R19.1, T10.B
- new net PHOTOTRANSISTOR: IC1.(T0/XCK)PB0, T7.C
- net ANODE1: no longer LED1.C@2
- net ANODE2: no longer LED2.C@2
- net ANODE3: no longer LED3.C@2
- net ANODE4: no longer LED4.C@2
- net VCC: now also D1.C, R14.1, R18.1, SP1.2, T5.C, T8.C
Other:
- note added: "Fake circuit with another phototransitor."
- moved on the sheet: LED1, LED2, LED3, LED4, T1, T2, T3, T4

Commit message: This time for sure schema is finished!
Parts:
- added S2: 5511, switch:5511
Connections:
- new net SECRET: IC1.(AIN0/INT2)PB2, S2.1A, S2.1B
- net GND: now also S2.NC, S2.NO
Other:
- note added: "Optional - to change between languages: 1. Elvish (default - custom numerals) 2. Common (arabic numerals)"
- moved on the sheet: S1, T2
